File: hardware/electronics/moss-core-v0.7/electrical/01_USB_Power.kicad_sch (KiCad schematic)
At the start: 24 parts, among them J1 USB2 device / 500mA max, U2 TPD2E2U06DCKR, U3 TPS2553DBVR, U4 TLV62569DBVR

Commit message: Update MOSS Core V0.7 prototype files for 31 October
Parts:
- U2: value TPD2E2U06DCKR -> TPD2E2U06QDCKRQ1; symbol MOSS:U2_TPD2E2U06DCKR -> MOSS:U2_TPD2E2U06QDCKRQ1; MPN TPD2E2U06DCKR -> TPD2E2U06QDCKRQ1
