File: hardware/electronics/moss-core-v0.7/electrical/16_Orange_Pi_Power.kicad_sch (KiCad schematic)
At the start: 8 parts, among them J20 5V3A OUT TO ORANGE PI, U42 TPS25810RVCR / USB-C source3A

Commit message: Update MOSS Core V0.7 prototype files for 31 October
Parts:
- removed MOD1: DC5-36-TO-DC3V3-5 / 5V, MOSS:MOSS_Power_Waveshare_DC5_36_TO_DC3V3_5_SMD_33x16mm_HandSolder, symbol MOSS:MOD1_DC5_36_TO_DC3V3_5___5V
- added C160: 22uF / 25V X7R, MOSS:Capacitor_SMD_C_1210_3225Metric, symbol MOSS:C160_22uF___25V_X7R
- added C162: 100nF / 50V X7R, MOSS:Capacitor_SMD_C_0603_1608Metric, symbol MOSS:C162_100nF___50V_X7R
- added C163: 100nF / 50V X7R, MOSS:Capacitor_SMD_C_0603_1608Metric, symbol MOSS:C163_100nF___50V_X7R
- added C164: 22uF / 10V X7R, MOSS:Capacitor_SMD_C_1206_3216Metric, symbol MOSS:C164_22uF___10V_X7R
- added C165: 22uF / 10V X7R, MOSS:Capacitor_SMD_C_1206_3216Metric, symbol MOSS:C165_22uF___10V_X7R
- added C166: 1uF / 10V, MOSS:Capacitor_SMD_C_0603_1608Metric, symbol MOSS:C166_1uF___10V
- added C167: 100nF / 50V X7R, MOSS:Capacitor_SMD_C_0603_1608Metric, symbol MOSS:C167_100nF___50V_X7R
- added C168: 33nF / 50V X7R, MOSS:Capacitor_SMD_C_0603_1608Metric, symbol MOSS:C168_33nF___50V_X7R
- added C169: 390pF / C0G, MOSS:Capacitor_SMD_C_0603_1608Metric, symbol MOSS:C169_390pF___C0G
- added L3: 10uH, MOSS:Inductor_SMD_L_Bourns_SRP6060FA, symbol MOSS:L3_10uH
- added R210: 499k, MOSS:Resistor_SMD_R_0603_1608Metric, symbol MOSS:R210_499k
- added R211: 100k, MOSS:Resistor_SMD_R_0603_1608Metric, symbol MOSS:R211_100k
- added R212: 4.7, MOSS:Resistor_SMD_R_0603_1608Metric, symbol MOSS:R212_4_7
- added R213: 53.6k, MOSS:Resistor_SMD_R_0603_1608Metric, symbol MOSS:R213_53_6k
- added R214: 10k, MOSS:Resistor_SMD_R_0603_1608Metric, symbol MOSS:R214_10k
- added R215: 845k, MOSS:Resistor_SMD_R_0603_1608Metric, symbol MOSS:R215_845k
- added U60: MP9447GL-Z / integrated host buck, MOSS:MOSS_Power_MP9447_QFN25_3x4, symbol MOSS:U60_MP9447GL_Z___integrated_host_buck
Connections:
- net GND: now also C160.2, C162.2, C163.2, C164.2, C165.2, C166.2, C168.2, R211.2, R214.2, U60.1 (AGND), U60.11 (PGND), U60.12 (PGND), U60.13 (PGND), U60.14 (PGND), U60.15 (PGND), U60.16 (PGND)
- net HOST_BUCK_IN: now also C160.1, C162.1, C163.1, R210.1, U60.19 (IN), U60.21 (IN), U60.22 (IN), U60.23 (IN), U60.8 (IN)
- net V5_HOST_RAW: now also C164.1, C165.1, L3.2, R213.1
- new net HOST_BST: R212.1, U60.7 (BST)
- new net HOST_BST_CAP: C167.1, R212.2
- new net HOST_EN: R210.2, U60.5 (EN)
- new net HOST_FB: C169.2, R213.2, R214.1, U60.3 (FB)
- new net HOST_FREQ: R211.1, U60.2 (FREQ)
- new net HOST_RAMP: C169.1, R215.2
- new net HOST_SS: C168.1, U60.4 (SS)
- new net HOST_SW: C167.2, L3.1, R215.1, U60.10 (SW), U60.17 (SW), U60.18 (SW), U60.24 (SW), U60.25 (SW), U60.9 (SW)
- new net HOST_VCC: C166.1, U60.20 (VCC)
- no-connect marks 12 -> 13
Other:
- note added: "3S battery -> F1 -> U60/L3 -> V5_HOST_RAW -> U42 -> HOST_5V -> J20. Keep VBUS and V5 separate."
- note added: "INTEGRATED HOST POWER / MP9447 / ENGINEERING CANDIDATE"
- note removed: "16 Orange Pi Power"
- note removed: "Power-only output to Orange Pi"
- note removed: "Replaceable input fuse and soldered5V module"
- note removed: "Soldered Waveshare5Vmodule andcompact3.15ASMDinputfuse. USB-CsourceCC/attach/switch control. Never bridge host output to USBdeviceVBUS."
- note removed: "USB-C source / attach switch / reference"
- title: MOSS Core V0.7 PROTOTYPE / 16 Orange Pi Power -> MOSS Core V0.7 PROTOTYPE / Integrated host supply
- moved on the sheet: C140, C141, C142, F1, J20, R200, U42
