File: hardware/electronics/moss-core-v0.7/electrical/04_Drive_Encoders.kicad_sch (KiCad schematic)
At the start: 44 parts, among them J2 CYTRON MDD10A SIGNAL, J3 ENCODER LEFT, J4 ENCODER RIGHT, U11 74LV08APWJ, U12 SN74LVC14APWR, U22 TPS22918DBVR

Commit message: Simplify MOSS Core motor harness connections
Parts:
- J2: value CYTRON MDD10A SIGNAL -> CYTRON LINK; footprint MOSS:Connector_JST_JST_GH_SM05B-GHS-TB_1x05-1MP_P1.25mm_Horizontal -> MOSS:Connector_Molex_Molex_Micro-Fit_3.0_43045-1012_2x05_P3.00mm_Vertical; symbol MOSS:J2_CYTRON_MDD10A_SIGNAL -> MOSS:J2_CYTRON_LINK; MPN SM05B-GHS-TB(LF)(SN) -> 43045-1012
- J3: value ENCODER LEFT -> LEFT MOTOR + ENCODER; footprint MOSS:Connector_JST_JST_GH_SM04B-GHS-TB_1x04-1MP_P1.25mm_Horizontal -> MOSS:Connector_Molex_Molex_Micro-Fit_3.0_43045-0612_2x03_P3.00mm_Vertical; symbol MOSS:J3_ENCODER_LEFT -> MOSS:J3_LEFT_MOTOR___ENCODER; MPN SM04B-GHS-TB(LF)(SN) -> 43045-0612
- J4: value ENCODER RIGHT -> RIGHT MOTOR + ENCODER; footprint MOSS:Connector_JST_JST_GH_SM04B-GHS-TB_1x04-1MP_P1.25mm_Horizontal -> MOSS:Connector_Molex_Molex_Micro-Fit_3.0_43045-0612_2x03_P3.00mm_Vertical; symbol MOSS:J4_ENCODER_RIGHT -> MOSS:J4_RIGHT_MOTOR___ENCODER; MPN SM04B-GHS-TB(LF)(SN) -> 43045-0612
Connections:
- net EL_A_EXT: now also J3.5 (ENC_A); no longer J3.3 (EL_A_EXT)
- net EL_B_EXT: now also J3.6 (ENC_B); no longer J3.4 (EL_B_EXT)
- net ENC_3V3: now also J3.4 (ENC_3V3), J4.4 (ENC_3V3); no longer J3.2 (ENC_3V3), J4.2 (ENC_3V3)
- net ER_A_EXT: now also J4.5 (ENC_A); no longer J4.3 (ER_A_EXT)
- net ER_B_EXT: now also J4.6 (ENC_B); no longer J4.4 (ER_B_EXT)
- net GND: now also J3.3 (ENC_GND), J4.3 (ENC_GND); no longer J2.MP (MOUNT), J3.1 (GND), J3.MP (MOUNT), J4.1 (GND), J4.MP (MOUNT)
- new net CYTRON_L_LEAD: J2.6 (LEFT_A)
- new net CYTRON_R_LEAD: J2.8 (RIGHT_A)
- new net MOTOR_L_LEAD: J3.1 (M1)
- new net MOTOR_L_RETURN: J2.7 (LEFT_B), J3.2 (M2)
- new net MOTOR_R_LEAD: J4.1 (M1)
- new net MOTOR_R_RETURN: J2.9 (RIGHT_B), J4.2 (M2)
- no-connect marks 2 -> 3
Other:
- note added: "MOSS CORE V0.7 / SIMPLIFIED MOTOR HARNESS / 31 OCTOBER 2026"
- note added: "One six-wire cable per motor. J2 to Cytron: four bridge outputs + PWM/DIR controls. Supply separately on J11."
- note removed: "04 Drive Encoders"
- note removed: "Cytron logic outputs: no motor power"
- note removed: "Encoder Schmitt receivers"
- note removed: "Encoder supply OFF until USB configured"
- note removed: "External CytronMDD10A PWM/DIR control and two encoder interfaces. No motor power inside the logic connector."
- note removed: "Left encoder / filters / ESD"
- note removed: "Motor request defaults and PWM mask"
- note removed: "Right encoder / filters / ESD"
- title: MOSS Core V0.7 PROTOTYPE / 04 Drive Encoders -> MOSS Core V0.7 PROTOTYPE / 04_Drive_Encoders
- moved on the sheet: C18, C19, C20, C21, C22, C23, C43, C44, C45, D6, D7, D8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
