File: hardware/electronics/moss-core-v0.7/electrical/17_Motor_Current.kicad_sch (KiCad schematic)
At the start: 16 parts, among them J12 L MOTOR SENSE LOOP, J13 R MOTOR SENSE LOOP, U40 INA240A2PWR, U41 INA240A2PWR, U43 ADS1115IDGSR

Commit message: Simplify MOSS Core motor harness connections
Parts:
- removed J12: L MOTOR SENSE LOOP, MOSS:TerminalBlock_Phoenix_TerminalBlock_Phoenix_MKDS-1,5-2-5.08_1x02_P5.08mm_Horizontal, symbol MOSS:J12_L_MOTOR_SENSE_LOOP
- removed J13: R MOTOR SENSE LOOP, MOSS:TerminalBlock_Phoenix_TerminalBlock_Phoenix_MKDS-1,5-2-5.08_1x02_P5.08mm_Horizontal, symbol MOSS:J13_R_MOTOR_SENSE_LOOP
Other:
- note added: "Existing INA240 and 2mR shunts retained. Motor-output legs are not GND. J12/J13 replaced by consolidated J2/J3/J4."
- note added: "MOSS CORE V0.7 / SIMPLIFIED MOTOR HARNESS / 31 OCTOBER 2026"
- note removed: "17 Motor Current"
- note removed: "Digital ADC and reference supply measurement"
- note removed: "Left in-line winding current"
- note removed: "Right in-line winding current"
- note removed: "Separate left/right in-linebidirectional motor currents; two shunts andPWM-rejecting amplifiers. ValidateADCcalibration,transients and thermal performance."
- title: MOSS Core V0.7 PROTOTYPE / 17 Motor Current -> MOSS Core V0.7 PROTOTYPE / 17_Motor_Current
- moved on the sheet: C120, C121, C122, C123, C124, C125, C126, R180, R181, R182, R183, U40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
