File: hardware/electronics/moss-core-v0.7/electrical/MOSS_Core_V07_Prototype.kicad_pcb (KiCad board)
At the start: 4 copper layers, 80 x 75 mm, 208 parts, among them J1 USB2 device / 500mA max, J10 XT30PW-M / FUSED 3S INPUT, J11 CYTRON POWER, J12 L MOTOR SENSE LOOP, J13 R MOTOR SENSE LOOP, J14 FAN 1 / 3S, J15 FAN 2 / 3S, J2 CYTRON MDD10A SIGNAL, J20 5V3A OUT TO ORANGE PI, J3 ENCODER LEFT, J4 ENCODER RIGHT, J5 ARM / DATA V+ GND, J7 SPEAKER / 4 ohm 3 W, J8 E-STOP / SIGNAL ONLY, Q2 MMBT3904, Q50 SiRA99DP, Q51 BSS138BK, Q52 BSS138BK, SW1 RESET_N, SW2 BOOT_N, U1 ESP32-S3-WROOM-1U-N8, U11 74LV08APWJ, U12 SN74LVC14APWR, U14 SN74LVC2G126DCUR, U15 SN74LVC1G126DCKR, U16 SN74LVC125APWR, U17 INA226 / BAT VOLTAGE, U2 TPD2E2U06DCKR, U20 TPS3808G33DBVR, U22 TPS22918DBVR, U23 MAX98357AETE+T, U24 TPS54302DDCR, U27 TPS3808G01DBVR, U3 TPS2553DBVR, U4 TLV62569DBVR, U40 INA240A2PWR, U41 INA240A2PWR, U42 TPS25810RVCR / USB-C source3A, U43 ADS1115IDGSR, U5 TPS3431SDRBR, U50 SN74LVC1G14, U6 SN74HCS21PWR

Commit message: Update MOSS Core V0.7 prototype files for 31 October
Parts:
- removed MOD1: DC5-36-TO-DC3V3-5 / 5V, MOSS:MOSS_Power_Waveshare_DC5_36_TO_DC3V3_5_SMD_33x16mm_HandSolder
- added C160: 22uF / 25V X7R, MOSS:Capacitor_SMD_C_1210_3225Metric, F.Cu at (42.0, 18.0)
- added C162: 100nF / 50V X7R, MOSS:Capacitor_SMD_C_0603_1608Metric, F.Cu at (39.1, 25.0)
- added C163: 100nF / 50V X7R, MOSS:Capacitor_SMD_C_0603_1608Metric, F.Cu at (32.0, 25.3)
- added C164: 22uF / 10V X7R, MOSS:Capacitor_SMD_C_1206_3216Metric, F.Cu at (42.3, 30.3)
- added C165: 22uF / 10V X7R, MOSS:Capacitor_SMD_C_1206_3216Metric, F.Cu at (36.9, 29.8)
- added C166: 1uF / 10V, MOSS:Capacitor_SMD_C_0603_1608Metric, F.Cu at (39.1, 21.5)
- added C167: 100nF / 50V X7R, MOSS:Capacitor_SMD_C_0603_1608Metric, F.Cu at (28.4, 21.3)
- added C168: 33nF / 50V X7R, MOSS:Capacitor_SMD_C_0603_1608Metric, F.Cu at (27.0, 29.0)
- added C169: 390pF / C0G, MOSS:Capacitor_SMD_C_0603_1608Metric, F.Cu at (32.0, 18.7)
- added L3: 10uH, MOSS:Inductor_SMD_L_Bourns_SRP6060FA, F.Cu at (43.5, 25.5)
- added R210: 499k, MOSS:Resistor_SMD_R_0603_1608Metric, F.Cu at (22.0, 25.0)
- added R211: 100k, MOSS:Resistor_SMD_R_0603_1608Metric, F.Cu at (37.4, 19.7)
- added R212: 4.7, MOSS:Resistor_SMD_R_0603_1608Metric, F.Cu at (31.5, 21.3)
- added R213: 53.6k, MOSS:Resistor_SMD_R_0603_1608Metric, F.Cu at (35.0, 17.1)
- added R214: 10k, MOSS:Resistor_SMD_R_0603_1608Metric, F.Cu at (35.0, 19.6)
- added R215: 845k, MOSS:Resistor_SMD_R_0603_1608Metric, F.Cu at (28.6, 18.7)
- added U60: MP9447GL-Z / integrated host buck, MOSS:MOSS_Power_MP9447_QFN25_3x4, F.Cu at (35.8, 25.0)
- H1: value M2.5 / drill 2.7 / keepout D8 -> M2.5 GND bond / drill2.7; footprint MOSS:MOSS_Mount_M2p5_2p7_D8 -> MOSS:MOSS_Mount_M2p5_GND_D8
- U2: value TPD2E2U06DCKR -> TPD2E2U06QDCKRQ1
Routing:
- net V5_HOST_RAW: track 33.1 -> 82.6 mm, vias 0 -> 7
- net PWM_L: track 92.2 -> 46.5 mm, vias 7 -> 6
- net HOST_BUCK_IN: track 124.5 -> 161.9 mm, vias 3 -> 6
- net HOST_SS: track 0.00 -> 30.4 mm
- net ER_A_F: track 134.0 -> 105.4 mm, vias 5 -> 6
- net HOST_SW: track 0.00 -> 26.2 mm
- net HOST_EN: track 0.00 -> 17.1 mm, vias 0 -> 2
- net MDD_DIR2: track 65.0 -> 79.4 mm, vias 6 -> 8
- net ESTOP_ACTIVE: track 71.9 -> 84.6 mm, vias 5 -> 7
- net GND: track 202.9 -> 214.7 mm, vias 142 -> 156
- net HOST_FB: track 0.00 -> 11.1 mm
- net AMP_ENABLE: track 79.8 -> 68.8 mm
- net ER_B_F: track 116.3 -> 122.9 mm, vias 6 -> 9
- net HOST_BST: track 0.00 -> 4.09 mm
- net HOST_FREQ: track 0.00 -> 3.38 mm
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Other:
- board text added: "GND"

Commit message: Simplify MOSS Core motor harness connections
Parts:
- removed J12: L MOTOR SENSE LOOP, MOSS:TerminalBlock_Phoenix_TerminalBlock_Phoenix_MKDS-1,5-2-5.08_1x02_P5.08mm_Horizontal
- removed J13: R MOTOR SENSE LOOP, MOSS:TerminalBlock_Phoenix_TerminalBlock_Phoenix_MKDS-1,5-2-5.08_1x02_P5.08mm_Horizontal
- J2: value CYTRON MDD10A SIGNAL -> CYTRON LINK; footprint MOSS:Connector_JST_JST_GH_SM05B-GHS-TB_1x05-1MP_P1.25mm_Horizontal -> MOSS:Connector_Molex_Molex_Micro-Fit_3.0_43045-1012_2x05_P3.00mm_Vertical
- J3: value ENCODER LEFT -> LEFT MOTOR + ENCODER; footprint MOSS:Connector_JST_JST_GH_SM04B-GHS-TB_1x04-1MP_P1.25mm_Horizontal -> MOSS:Connector_Molex_Molex_Micro-Fit_3.0_43045-0612_2x03_P3.00mm_Vertical
- J4: value ENCODER RIGHT -> RIGHT MOTOR + ENCODER; footprint MOSS:Connector_JST_JST_GH_SM04B-GHS-TB_1x04-1MP_P1.25mm_Horizontal -> MOSS:Connector_Molex_Molex_Micro-Fit_3.0_43045-0612_2x03_P3.00mm_Vertical
- moved J3 69.1 mm to (3.00, 44.0), turned to 0 degrees
- moved J8 64.5 mm to (60.0, 5.00), turned to 0 degrees
- moved J4 59.6 mm to (3.00, 55.4), turned to 0 degrees
- moved J2 11.6 mm to (34.5, 1.30), turned to 0 degrees
Connections:
- J3 pad 1: GND -> MOTOR_L_LEAD
- J3 pad 2: ENC_3V3 -> MOTOR_L_RETURN
- J3 pad 3: EL_A_EXT -> GND
- J3 pad 4: EL_B_EXT -> ENC_3V3
- J4 pad 1: GND -> MOTOR_R_LEAD
- J4 pad 2: ENC_3V3 -> MOTOR_R_RETURN
- J4 pad 3: ER_A_EXT -> GND
- J4 pad 4: ER_B_EXT -> ENC_3V3
Routing:
- net CYTRON_R_LEAD: track 29.8 -> 114.1 mm, vias 8 -> 12
- net ENC_3V3: track 125.7 -> 208.0 mm, vias 4 -> 18
- net ESTOP_CUT_SOURCE: track 21.5 -> 101.6 mm, vias 1 -> 12
- net MOTOR_R_RETURN: track 0.00 -> 79.5 mm, vias 0 -> 9
- net EL_B_EXT: track 11.8 -> 77.9 mm, vias 0 -> 2
- net EL_A_EXT: track 16.6 -> 79.9 mm, vias 0 -> 3
- net MOTOR_L_RETURN: track 0.00 -> 60.9 mm, vias 0 -> 3
- net MDD_DIR2: track 79.4 -> 27.2 mm, vias 8 -> 2
- net ESTOP_STATUS_RAW: track 40.5 -> 92.7 mm, vias 1 -> 16
- net AMP_ENABLE: track 68.8 -> 117.7 mm, vias 5 -> 13
- net ER_B_EXT: track 27.7 -> 70.6 mm, vias 1 -> 0
- net ESTOP_CUT_RETURN: track 21.7 -> 63.0 mm, vias 1 -> 5
- net CYTRON_L_LEAD: track 31.7 -> 69.8 mm
- net ESTOP_STATUS_SOURCE: track 21.3 -> 54.3 mm, vias 1 -> 3
- net ER_A_EXT: track 25.9 -> 51.7 mm, vias 1 -> 2
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Other:
- board size 80 x 75 mm -> 82 x 75 mm
- board text added: "J2 CYTRON LINK 1 PWM1 | 2 DIR1 | 3 PWM2 | 4 DIR2 | 5 GND 6 LA | 7 LB | 8 RA | 9 RB | 10 NO WIRE"
- board text added: "J3 LEFT MOTOR 1 M1 | 2 M2 | 3 GND 4 3V3 | 5 A | 6 B"
- board text added: "J4 RIGHT MOTOR 1 M1 | 2 M2 | 3 GND 4 3V3 | 5 A | 6 B"
- board text removed: "J12 LEFT MOTOR 1 CYTRON 2 MOTOR"
- board text removed: "J13 RIGHT MOTOR 1 CYTRON 2 MOTOR"
- board text removed: "J2 CYTRON CTRL 1 PWM1 | 2 DIR1 3 PWM2 | 4 DIR2 | 5 GND"
- board text removed: "J3 ENC LEFT 1 GND | 2 3V3 3 A | 4 B"
- board text removed: "J4 ENC RIGHT 1 GND | 2 3V3 3 A | 4 B"
